Commit message: fifth checkpoint

File: urdf/robot.urdf (robot description, URDF)
Before this commit: robot myRobot, 4 links, 3 joints
Links:
- removed link big_head
- removed link left_leg
- removed link middle_hand
- added link forth_segment; collision cylinder length=0.9 radius=0.12; visual cylinder length=0.9 radius=0.12
- added link gripper_base; collision box size=0.3 0.4 0.03; visual box size=0.3 0.4 0.03
- added link left_gripper; collision box size=0.3 0.03 0.2; visual box size=0.3 0.03 0.2
- added link right_gripper; collision box size=0.3 0.03 0.2; visual box size=0.3 0.03 0.2
- added link second_segment; collision cylinder length=0.3 radius=0.25; visual cylinder length=0.3 radius=0.25
- added link third_segment; collision cylinder length=0.9 radius=0.15; visual cylinder length=0.9 radius=0.15
- link base_link: geometry collision cylinder length=0.8 radius=0.2; visual cylinder length=0.8 radius=0.2
Joints:
- removed joint big_head_joint
- removed joint left_leg_joint
- removed joint right_leg_joint
- added joint forth_segment_joint: type revolute, parent third_segment, child forth_segment, origin xyz=0 0 0.9, axis 0 1 0, limit lower=-0.4 upper=1.2 effort=1000.0 velocity=0.5
- added joint gripper_joint: type fixed, parent forth_segment, child gripper_base, origin xyz=0 0 0.9
- added joint left_gripper_joint: type prismatic, parent gripper_base, child left_gripper, origin xyz=0 0 0.015, axis 0 1 0, limit lower=-0.06 upper=0.06 effort=1000 velocity=0.5
- added joint right_gripper_joint: type prismatic, parent gripper_base, child right_gripper, origin xyz=0 0 0.015, axis 0 1 0, limit lower=-0.06 upper=0.06 effort=1000 velocity=0.5
- added joint second_segment_joint: type revolute, parent base_link, child second_segment, origin xyz=0 0 0.8, axis 0 0 1, limit lower=-0.4 upper=2 effort=1000.0 velocity=0.5
- added joint third_segment_joint: type revolute, parent second_segment, child third_segment, origin xyz=0 0 0.3, axis 0 1 0, limit lower=-0.4 upper=1.2 effort=1000.0 velocity=0.5
